File: CAN.sch (KiCad schematic (older format))
At the start: 6 parts, among them P2 CONN_01X03, U3 SN65HVD232

Commit message: - #4 Added UART and CAN interface transceivers - Improved schematic structure - Removed all gerber outputs - Generated schematics outputs for PCB design - Updated local libraries
Parts:
- C18: footprint ~ -> Capacitors_SMD:C_0805_HandSoldering
- C19: footprint ~ -> Capacitors_SMD:C_0603_HandSoldering
- JP2: footprint (none) -> ComponentLibv2:AYZ-SlideSwitches
- P2: footprint (none) -> Pin_Headers:Pin_Header_Straight_1x03
- R15: footprint ~ -> Resistors_SMD:R_0805_HandSoldering
- U3: footprint (none) -> Housings_SOIC:SOIC-8_3.9x4.9mm_Pitch1.27mm
Changed lines of the file:
@@
 F 0 "U3" H 5950 4450 60  0000 C CNN
 F 1 "SN65HVD232" H 5950 5050 60  0000 C CNN
-F 2 "" H 5950 4750 60  0000 C CNN
+F 2 "Housings_SOIC:SOIC-8_3.9x4.9mm_Pitch1.27mm" H 5950 4750 60  0001 C CNN
 F 3 "" H 5950 4750 60  0000 C CNN
 	1    5950 4750
@@
 F 0 "C19" H 6150 4000 40  0000 L CNN
 F 1 "100n" H 6156 3815 40  0000 L CNN
-F 2 "~" H 6188 3750 30  0000 C CNN
+F 2 "Capacitors_SMD:C_0603_HandSoldering" H 6188 3750 30  0001 C CNN
 F 3 "~" H 6150 3900 60  0000 C CNN
 	1    6150 3900
@@
 F 0 "R15" V 7280 4600 40  0000 C CNN
 F 1 "120" V 7207 4601 40  0000 C CNN
-F 2 "~" V 7130 4600 30  0000 C CNN
+F 2 "Resistors_SMD:R_0805_HandSoldering" V 7130 4600 30  0001 C CNN
 F 3 "~" H 7200 4600 30  0000 C CNN
 	1    7200 4600
@@
 F 0 "C18" H 5800 4000 40  0000 L CNN
 F 1 "10u" H 5806 3815 40  0000 L CNN
-F 2 "~" H 5838 3750 30  0000 C CNN
+F 2 "Capacitors_SMD:C_0805_HandSoldering" H 5838 3750 30  0001 C CNN
 F 3 "~" H 5800 3900 60  0000 C CNN
 	1    5800 3900
@@
 F 0 "JP2" H 7200 5180 50  0000 C CNN
 F 1 "Jumper_NC_Small" H 7210 5040 50  0001 C CNN
-F 2 "" H 7200 5100 60  0000 C CNN
+F 2 "ComponentLibv2:AYZ-SlideSwitches" H 7200 5100 60  0001 C CNN
 F 3 "" H 7200 5100 60  0000 C CNN
 	1    7200 5100
@@
 F 0 "P2" H 8350 5000 50  0000 C CNN
 F 1 "CONN_01X03" V 8450 4800 50  0000 C CNN
-F 2 "" H 8350 4800 60  0000 C CNN
+F 2 "Pin_Headers:Pin_Header_Straight_1x03" H 8350 4800 60  0001 C CNN
 F 3 "" H 8350 4800 60  0000 C CNN
 	1    8350 4800
