File: Clocks.sch (KiCad schematic (older format))
At the start: 5 parts, among them X1 25 MHz

Commit message: - #4 Added UART and CAN interface transceivers - Improved schematic structure - Removed all gerber outputs - Generated schematics outputs for PCB design - Updated local libraries
Parts:
- C16, C17: footprint ~ -> Capacitors_SMD:C_0603_HandSoldering
- R13, R14: footprint ~ -> Resistors_SMD:R_0603_HandSoldering
- X1: footprint ~ -> ComponentLibv2:7A-25.000MAAJ-T
Changed lines of the file:
@@
 F 0 "X1" H 5850 4950 60  0000 C CNN
 F 1 "25 MHz" H 5850 4650 60  0000 C CNN
-F 2 "~" H 5850 4800 60  0000 C CNN
-F 3 "~" H 5850 4800 60  0000 C CNN
+F 2 "ComponentLibv2:7A-25.000MAAJ-T" H 5850 4800 60  0001 C CNN
+F 3 "http://www.farnell.com/datasheets/1041607.pdf" H 5850 4800 60  0001 C CNN
 	1    5850 4800
 	0    -1   -1   0
@@
 F 0 "C16" H 5550 4600 40  0000 L CNN
 F 1 "4.7p" H 5556 4415 40  0000 L CNN
-F 2 "~" H 5588 4350 30  0000 C CNN
+F 2 "Capacitors_SMD:C_0603_HandSoldering" H 5588 4350 30  0001 C CNN
 F 3 "~" H 5550 4500 60  0000 C CNN
 	1    5550 4500
@@
 F 0 "C17" H 5550 5200 40  0000 L CNN
 F 1 "4.7p" H 5556 5015 40  0000 L CNN
-F 2 "~" H 5588 4950 30  0000 C CNN
+F 2 "Capacitors_SMD:C_0603_HandSoldering" H 5588 4950 30  0001 C CNN
 F 3 "~" H 5550 5100 60  0000 C CNN
 	1    5550 5100
@@
 F 0 "R13" V 6280 4500 40  0000 C CNN
 F 1 "0" H 6207 4501 40  0000 C CNN
-F 2 "~" V 6130 4500 30  0000 C CNN
+F 2 "Resistors_SMD:R_0603_HandSoldering" V 6130 4500 30  0001 C CNN
 F 3 "~" H 6200 4500 30  0000 C CNN
 	1    6200 4500
@@
 F 0 "R14" V 6280 5100 40  0000 C CNN
 F 1 "0" H 6207 5101 40  0000 C CNN
-F 2 "~" V 6130 5100 30  0000 C CNN
+F 2 "Resistors_SMD:R_0603_HandSoldering" V 6130 5100 30  0001 C CNN
 F 3 "~" H 6200 5100 30  0000 C CNN
 	1    6200 5100
