File: Debug.sch (KiCad schematic (older format))
At the start: 2 parts, among them CON1 SWD

Commit message: - #4 Added UART and CAN interface transceivers - Improved schematic structure - Removed all gerber outputs - Generated schematics outputs for PCB design - Updated local libraries
Parts:
- CON1: footprint (none) -> Pin_Headers:Pin_Header_Straight_1x06
- JP1: footprint (none) -> Resistors_SMD:R_0603_HandSoldering
Changed lines of the file:
@@
 F 0 "CON1" H 5350 5300 60  0000 C CNN
 F 1 "SWD" H 5350 4500 60  0000 C CNN
-F 2 "" H 5550 4900 60  0000 C CNN
+F 2 "Pin_Headers:Pin_Header_Straight_1x06" H 5550 4900 60  0001 C CNN
 F 3 "" H 5550 4900 60  0000 C CNN
 	1    5550 4900
@@
 F 0 "JP1" H 5950 5050 50  0000 C CNN
 F 1 "Jumper_NO_Small" H 5960 5090 50  0001 C CNN
-F 2 "" H 5950 5150 60  0000 C CNN
+F 2 "Resistors_SMD:R_0603_HandSoldering" H 5950 5150 60  0001 C CNN
 F 3 "" H 5950 5150 60  0000 C CNN
 	1    5950 5150
