File: MCU.sch (KiCad schematic (older format))
At the start: 15 parts, among them U6 STM32F405RGT6

Commit message: - #4 Added UART and CAN interface transceivers - Improved schematic structure - Removed all gerber outputs - Generated schematics outputs for PCB design - Updated local libraries
Parts:
- C25, C26, C33: footprint ~ -> Capacitors_SMD:C_0805_HandSoldering
- C27, C28, C29, C30, C31, C32: footprint ~ -> Capacitors_SMD:C_0603_HandSoldering
- JP3, JP4, R22, R23: footprint (none) -> Resistors_SMD:R_0603_HandSoldering
- R24: footprint ~ -> Resistors_SMD:R_0603_HandSoldering
- U6: footprint ~ -> Housings_QFP:LQFP-64_10x10mm_Pitch0.5mm
Changed lines of the file:
@@
 F 0 "U6" H 9050 3300 60  0000 C CNN
 F 1 "STM32F405RGT6" H 9050 3500 60  0000 C CNN
-F 2 "~" H 8850 3400 60  0000 C CNN
+F 2 "Housings_QFP:LQFP-64_10x10mm_Pitch0.5mm" H 8850 3400 60  0001 C CNN
 F 3 "~" H 8850 3400 60  0000 C CNN
 	1    9050 3400
@@
 F 0 "C32" H 5900 6500 40  0000 L CNN
 F 1 "100n" H 5906 6315 40  0000 L CNN
-F 2 "~" H 5938 6250 30  0000 C CNN
+F 2 "Capacitors_SMD:C_0603_HandSoldering" H 5938 6250 30  0001 C CNN
 F 3 "~" H 5900 6400 60  0000 C CNN
 	1    5900 6400
@@
 F 0 "C30" H 5600 6500 40  0000 L CNN
 F 1 "100n" H 5606 6315 40  0000 L CNN
-F 2 "~" H 5638 6250 30  0000 C CNN
+F 2 "Capacitors_SMD:C_0603_HandSoldering" H 5638 6250 30  0001 C CNN
 F 3 "~" H 5600 6400 60  0000 C CNN
 	1    5600 6400
@@
 F 0 "C27" H 5000 6500 40  0000 L CNN
 F 1 "100n" H 5006 6315 40  0000 L CNN
-F 2 "~" H 5038 6250 30  0000 C CNN
+F 2 "Capacitors_SMD:C_0603_HandSoldering" H 5038 6250 30  0001 C CNN
 F 3 "~" H 5000 6400 60  0000 C CNN
 	1    5000 6400
@@
 F 0 "C29" H 5300 6500 40  0000 L CNN
 F 1 "100n" H 5306 6315 40  0000 L CNN
-F 2 "~" H 5338 6250 30  0000 C CNN
+F 2 "Capacitors_SMD:C_0603_HandSoldering" H 5338 6250 30  0001 C CNN
 F 3 "~" H 5300 6400 60  0000 C CNN
 	1    5300 6400
@@
 F 0 "C28" H 5300 2150 40  0000 L CNN
 F 1 "100n" H 5306 1965 40  0000 L CNN
-F 2 "~" H 5338 1900 30  0000 C CNN
+F 2 "Capacitors_SMD:C_0603_HandSoldering" H 5338 1900 30  0001 C CNN
 F 3 "~" H 5300 2050 60  0000 C CNN
 	1    5300 2050
@@
 F 0 "R24" V 5680 1850 40  0000 C CNN
 F 1 "47" V 5607 1851 40  0000 C CNN
-F 2 "~" V 5530 1850 30  0000 C CNN
+F 2 "Resistors_SMD:R_0603_HandSoldering" V 5530 1850 30  0001 C CNN
 F 3 "~" H 5600 1850 30  0000 C CNN
 	1    5600 1850
@@
 F 0 "C31" H 5900 2150 40  0000 L CNN
 F 1 "1u" H 5906 1965 40  0000 L CNN
-F 2 "~" H 5938 1900 30  0000 C CNN
+F 2 "Capacitors_SMD:C_0603_HandSoldering" H 5938 1900 30  0001 C CNN
 F 3 "~" H 5900 2050 60  0000 C CNN
 	1    5900 2050
@@
 F 0 "C25" H 4850 3900 50  0000 L CNN
 F 1 "2u2" H 4850 3700 50  0000 L CNN
-F 2 "~" H 4800 3800 60  0000 C CNN
+F 2 "Capacitors_SMD:C_0805_HandSoldering" H 4800 3800 60  0001 C CNN
 F 3 "~" H 4800 3800 60  0000 C CNN
 	1    4800 3800
@@
 F 0 "C26" H 4850 5000 50  0000 L CNN
 F 1 "2u2" H 4850 4800 50  0000 L CNN
-F 2 "~" H 4800 4900 60  0000 C CNN
+F 2 "Capacitors_SMD:C_0805_HandSoldering" H 4800 4900 60  0001 C CNN
 F 3 "~" H 4800 4900 60  0000 C CNN
 	1    4800 4900
@@
 F 0 "C33" H 6350 6500 50  0000 L CNN
 F 1 "4u7" H 6350 6300 50  0000 L CNN
-F 2 "~" H 6300 6400 60  0000 C CNN
+F 2 "Capacitors_SMD:C_0805_HandSoldering" H 6300 6400 60  0001 C CNN
 F 3 "~" H 6300 6400 60  0000 C CNN
 	1    6300 6400
@@
 F 0 "JP3" H 5300 4980 50  0000 C CNN
 F 1 "Jumper_NO_Small" H 5310 4840 50  0001 C CNN
-F 2 "" H 5300 4900 60  0000 C CNN
+F 2 "Resistors_SMD:R_0603_HandSoldering" H 5300 4900 60  0001 C CNN
 F 3 "" H 5300 4900 60  0000 C CNN
 	1    5300 4900
@@
 F 0 "JP4" H 5350 3830 50  0000 C CNN
 F 1 "Jumper_NO_Small" H 5360 3690 50  0001 C CNN
-F 2 "" H 5350 3750 60  0000 C CNN
+F 2 "Resistors_SMD:R_0603_HandSoldering" H 5350 3750 60  0001 C CNN
 F 3 "" H 5350 3750 60  0000 C CNN
 	1    5350 3750
@@
 F 0 "R22" V 1880 2600 50  0000 C CNN
 F 1 "0" V 1800 2600 50  0000 C CNN
-F 2 "" V 1730 2600 30  0000 C CNN
+F 2 "Resistors_SMD:R_0603_HandSoldering" V 1730 2600 30  0001 C CNN
 F 3 "" H 1800 2600 30  0000 C CNN
 	1    1800 2600
@@
 F 0 "R23" V 2130 2800 50  0000 C CNN
 F 1 "1K" V 2050 2800 50  0000 C CNN
-F 2 "" V 1980 2800 30  0000 C CNN
+F 2 "Resistors_SMD:R_0603_HandSoldering" V 1980 2800 30  0001 C CNN
 F 3 "" H 2050 2800 30  0000 C CNN
 	1    2050 2800
