File: SDIO.sch (KiCad schematic (older format))
At the start: 7 parts, among them U5 SD_CARD

Commit message: - #4 Added UART and CAN interface transceivers - Improved schematic structure - Removed all gerber outputs - Generated schematics outputs for PCB design - Updated local libraries
Parts:
- R16, R17, R18, R19, R20, R21: footprint (none) -> Resistors_SMD:R_0603_HandSoldering
- U5: footprint (none) -> ComponentLibv2:uSDCard
Changed lines of the file:
@@
 F 0 "U5" H 7600 3300 60  0000 C CNN
 F 1 "SD_CARD" H 7550 4300 60  0000 C CNN
-F 2 "" H 7300 3800 60  0000 C CNN
-F 3 "" H 7300 3800 60  0000 C CNN
+F 2 "ComponentLibv2:uSDCard" H 7300 3800 60  0001 C CNN
+F 3 "Molex - 502570-0893" H 7300 3800 60  0001 C CNN
 	1    7600 3800
 	1    0    0    -1
@@
 F 0 "R21" V 7530 5050 50  0000 C CNN
 F 1 "0" V 7450 5050 50  0000 C CNN
-F 2 "" V 7380 5050 30  0000 C CNN
+F 2 "Resistors_SMD:R_0603_HandSoldering" V 7380 5050 30  0001 C CNN
 F 3 "" H 7450 5050 30  0000 C CNN
 	1    7450 5050
@@
 F 0 "R16" V 3530 4400 50  0000 C CNN
 F 1 "47K" V 3450 4400 50  0000 C CNN
-F 2 "" V 3380 4400 30  0000 C CNN
+F 2 "Resistors_SMD:R_0603_HandSoldering" V 3380 4400 30  0001 C CNN
 F 3 "" H 3450 4400 30  0000 C CNN
 	1    3450 4400
@@
 F 0 "R17" V 3730 4400 50  0000 C CNN
 F 1 "47K" V 3650 4400 50  0000 C CNN
-F 2 "" V 3580 4400 30  0000 C CNN
+F 2 "Resistors_SMD:R_0603_HandSoldering" V 3580 4400 30  0001 C CNN
 F 3 "" H 3650 4400 30  0000 C CNN
 	1    3650 4400
@@
 F 0 "R18" V 3930 4400 50  0000 C CNN
 F 1 "47K" V 3850 4400 50  0000 C CNN
-F 2 "" V 3780 4400 30  0000 C CNN
+F 2 "Resistors_SMD:R_0603_HandSoldering" V 3780 4400 30  0001 C CNN
 F 3 "" H 3850 4400 30  0000 C CNN
 	1    3850 4400
@@
 F 0 "R19" V 4130 4400 50  0000 C CNN
 F 1 "47K" V 4050 4400 50  0000 C CNN
-F 2 "" V 3980 4400 30  0000 C CNN
+F 2 "Resistors_SMD:R_0603_HandSoldering" V 3980 4400 30  0001 C CNN
 F 3 "" H 4050 4400 30  0000 C CNN
 	1    4050 4400
@@
 F 0 "R20" V 4330 4400 50  0000 C CNN
 F 1 "47K" V 4250 4400 50  0000 C CNN
-F 2 "" V 4180 4400 30  0000 C CNN
+F 2 "Resistors_SMD:R_0603_HandSoldering" V 4180 4400 30  0001 C CNN
 F 3 "" H 4250 4400 30  0000 C CNN
 	1    4250 4400
