File: UART.sch (KiCad schematic (older format))
At the start: 7 parts, among them P3 CONN_01X03, U4 MAX232

Commit message: - #4 Added UART and CAN interface transceivers - Improved schematic structure - Removed all gerber outputs - Generated schematics outputs for PCB design - Updated local libraries
Parts:
- C20, C21, C22, C23, C24: footprint ~ -> Capacitors_SMD:C_0603_HandSoldering
- P3: footprint (none) -> Pin_Headers:Pin_Header_Straight_1x03
- U4: footprint (none) -> Housings_SOIC:SOIC-16_3.9x9.9mm_Pitch1.27mm
Changed lines of the file:
@@
 F 0 "C20" H 5200 3700 40  0000 L CNN
 F 1 "1u" H 5206 3515 40  0000 L CNN
-F 2 "~" H 5238 3450 30  0000 C CNN
+F 2 "Capacitors_SMD:C_0603_HandSoldering" H 5238 3450 30  0001 C CNN
 F 3 "~" H 5200 3600 60  0000 C CNN
 	1    5200 3600
@@
 F 0 "P3" H 7900 4700 50  0000 C CNN
 F 1 "CONN_01X03" V 8000 4500 50  0000 C CNN
-F 2 "" H 7900 4500 60  0000 C CNN
+F 2 "Pin_Headers:Pin_Header_Straight_1x03" H 7900 4500 60  0001 C CNN
 F 3 "" H 7900 4500 60  0000 C CNN
 	1    7900 4500
@@
 F 0 "C21" H 5200 4200 40  0000 L CNN
 F 1 "1u" H 5206 4015 40  0000 L CNN
-F 2 "~" H 5238 3950 30  0000 C CNN
+F 2 "Capacitors_SMD:C_0603_HandSoldering" H 5238 3950 30  0001 C CNN
 F 3 "~" H 5200 4100 60  0000 C CNN
 	1    5200 4100
@@
 F 0 "C24" H 7300 3700 40  0000 L CNN
 F 1 "1u" H 7306 3515 40  0000 L CNN
-F 2 "~" H 7338 3450 30  0000 C CNN
+F 2 "Capacitors_SMD:C_0603_HandSoldering" H 7338 3450 30  0001 C CNN
 F 3 "~" H 7300 3600 60  0000 C CNN
 	1    7300 3600
@@
 F 0 "C22" H 6850 3900 40  0000 L CNN
 F 1 "1u" H 6856 3715 40  0000 L CNN
-F 2 "~" H 6888 3650 30  0000 C CNN
+F 2 "Capacitors_SMD:C_0603_HandSoldering" H 6888 3650 30  0001 C CNN
 F 3 "~" H 6850 3800 60  0000 C CNN
 	1    6850 3800
@@
 F 0 "C23" H 6850 4400 40  0000 L CNN
 F 1 "1u" H 6856 4215 40  0000 L CNN
-F 2 "~" H 6888 4150 30  0000 C CNN
+F 2 "Capacitors_SMD:C_0603_HandSoldering" H 6888 4150 30  0001 C CNN
 F 3 "~" H 6850 4300 60  0000 C CNN
 	1    6850 4300
@@
 F 0 "U4" H 5450 4950 50  0000 L CNN
 F 1 "MAX232" H 6100 4950 50  0000 L CNN
-F 2 "" H 5900 4100 60  0000 C CNN
+F 2 "Housings_SOIC:SOIC-16_3.9x9.9mm_Pitch1.27mm" H 5900 4100 60  0001 C CNN
 F 3 "" H 5900 4100 60  0000 C CNN
 	1    5900 4100
